File: LabPS.kicad_pcb (KiCad board)
At the start: 2 copper layers, 57 parts, among them J1 Fan, J2 24Vac, J3 P2, J4 P1, J5 Vo, Q1 BC558, Q2 BD139, Q3 BC548, Q4 TIP3055, U1 L7812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

Commit message: Final PCB layout.
Parts:
- R3: footprint Resistor_THT:R_Axial_DIN0918_L18.0mm_D9.0mm_P30.48mm_Horizontal -> Resistor_THT:R_Axial_DIN0614_L14.3mm_D5.7mm_P15.24mm_Horizontal
- moved C2 98.8 mm to (151.9, 99.8), turned to 90 degrees
- moved D12 96.8 mm to (179.5, 64.3), turned to 180 degrees
- moved D4 80.6 mm to (129.9, 97.8), turned to 180 degrees
- moved D5 79.5 mm to (129.9, 105.4), turned to 180 degrees
- moved R5 71.8 mm to (127.4, 126.4)
- moved R14 70.9 mm to (188.5, 108.8), turned to 270 degrees
- moved Q1 63.5 mm to (122.2, 129.7), turned to 90 degrees
- moved J2 63.5 mm to (114.7, 75.3)
- moved Q2 61.1 mm to (136.1, 63.9)
- moved J4 60.4 mm to (171.2, 130.3), turned to 270 degrees
- moved R20 54.7 mm to (157.7, 83.2)
- moved R12 54.2 mm to (174.6, 126.4)
- moved U2 54.0 mm to (152.9, 118.5), turned to 180 degrees
- moved J1 53.0 mm to (124.8, 69.8)
- moved C3 52.8 mm to (133.2, 117.5), turned to 180 degrees
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Connections:
- J2 pad 1: Net-(D3-Pad1) -> Net-(D2-Pad1)
- J2 pad 2: Net-(D2-Pad1) -> Net-(D3-Pad1)
Routing:
- net Net-(C2-Pad1): track 0.00 -> 236.9 mm, vias 0 -> 4
- net Net-(D8-Pad2): track 0.00 -> 200.9 mm, vias 0 -> 3
- net Net-(C5-Pad1): track 0.00 -> 194.6 mm
- net Net-(C2-Pad2): track 0.00 -> 155.4 mm, vias 0 -> 2
- net Net-(C8-Pad2): track 0.00 -> 126.8 mm
- net Net-(C6-Pad1): track 0.00 -> 91.5 mm
- net Net-(C6-Pad2): track 0.00 -> 62.6 mm
- net Net-(C4-Pad2): track 0.00 -> 57.7 mm
- net Net-(D3-Pad1): track 0.00 -> 47.6 mm
- net Net-(D9-Pad2): track 0.00 -> 47.5 mm
- net Net-(Q3-Pad2): track 0.00 -> 45.8 mm
- net Net-(Q2-Pad1): track 0.00 -> 40.1 mm
- net Net-(C5-Pad2): track 0.00 -> 39.2 mm
- net Net-(R12-Pad2): track 0.00 -> 35.9 mm
- net Net-(D11-Pad1): track 0.00 -> 33.7 mm
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Other:
- board outline added: 84.8 x 76.3 mm
- board text added: "Kobaya 2020"
- board text added: "LabPS"
